File: TangPrimer25K_brushless.kicad_pcb (KiCad board)
At the start: 2 copper layers, 81.5 x 99.9 mm, 27 parts, among them CN1 Nucleo_F302R8, J2 01x08_Socket, J3 01x04_Socket, SW2 SW_SPDT, SW3 SW_SPDT, U1 Tang_Nano_9k_board, U2 MCP3008, U3 PinHeader_1x12_P2.54mm_Vertic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

Commit message: 0416
Parts:
- removed J2: 01x08_Socket, Connector_PinSocket_2.54mm:PinSocket_1x08_P2.54mm_Vertical
- removed J3: 01x04_Socket, Connector_PinSocket_2.54mm:PinSocket_1x04_P2.54mm_Vertical
- removed R10, R3, R4, R5, R6, R7, R8, R9: R, Resistor_SMD:R_0603_1608Metric_Pad0.98x0.95mm_HandSolder
- removed S1, S2, S3, S4: TVGP01-G73BB, SamacSys_Parts:TVGP01G73BB
- removed U1: Tang_Nano_9k_board, Library:Tang Nano 9K
- removed U3: PinHeader_1x12_P2.54mm_Vertical, Connector_PinHeader_2.54mm:PinHeader_1x12_P2.54mm_Vertical
Routing:
- net Net-(U1-25/IOB8A): track 83.3 -> 0.00 mm
- net Net-(U1-26/IOB8B): track 79.8 -> 0.00 mm
- net Net-(U1-27/IOB11A): track 76.4 -> 0.00 mm
- net Net-(SW1-B): track 74.7 -> 0.25 mm
- net /DIG1: track 73.8 -> 0.00 mm
- net Net-(U1-28/IOB11B): track 73.1 -> 0.00 mm
- net Net-(U1-29/IOB13A): track 69.7 -> 0.00 mm
- net /_LIN_S: track 87.8 -> 18.2 mm
- net /DIG3: track 68.0 -> 0.00 mm
- net /DIG2: track 64.8 -> 0.00 mm
- net Net-(U1-33/IOB23A/RGB_DE): track 63.5 -> 0.00 mm
- net Net-(SW2-B): track 81.4 -> 19.6 mm
- net /SW3: track 88.1 -> 31.3 mm
- net Net-(U1-35/IOB29A/RGB_CK): track 54.4 -> 0.00 mm
- net Net-(S1-NO_1): track 46.2 -> 0.00 mm
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Other:
- board text removed: "<HDMI>"
- board text removed: "<USB>"
- board text removed: "A"
- board text removed: "B"
- board text removed: "C"
- board text removed: "D"
- board text removed: "DIG1"
- board text removed: "DIG2"
- board text removed: "DIG3"
- board text removed: "DIG4"
- board text removed: "DP"
- board text removed: "E"
- board text removed: "F"
- board text removed: "G"
- board text removed: "[Tang Nano 9K]"

Commit message: 0416
Parts:
- removed G***: LOGO, MyLibrary:kamo20
- removed Reverse, SW2, SW3: SW_SPDT, Connector_PinHeader_2.54mm:PinHeader_1x03_P2.54mm_Vertical
- added J1: DF40C-60DS-0.4V_51_, Library:DF40C-60DS-0.4V_51_, F.Cu at (170.9, 118.2)
- added J2: DF40C-60DS-0.4V_51_, Library:DF40C-60DS-0.4V_51_, F.Cu at (153.3, 118.4)
- added S3: TVGP01-G73BB, SamacSys_Parts:TVGP01G73BB, F.Cu at (169.6, 161.2)
- added S4: TVGP01-G73BB, SamacSys_Parts:TVGP01G73BB, F.Cu at (148.6, 162.2)
- moved R1 71.8 mm to (146.9, 152.4), turned to 180 degrees
- moved R2 69.8 mm to (142.9, 152.9), turned to 180 degrees
- moved JP1 69.0 mm to (145.5, 149.8)
- moved C1 67.4 mm to (136.0, 149.4), turned to 180 degrees
- moved U2 58.4 mm to (139.7, 138.3), turned to -90 degrees
- renumbered CN1 to J3
Connections:
- J3 pad 66: /C10-28 -> unconnected-(J3-Pad66)
- J3 pad 68: unconnected-(J1-Pad68) -> /C7-30
- U2 pad 1: /C10-11 -> /C7-30
- U2 pad 12: Net-(U1-31/IOB15A/RGB_TOUCH_YD) -> unconnected-(U2-Dout-Pad12)
- U2 pad 13: Net-(U1-32/IOB15B/RGB_TOUCH_XR) -> unconnected-(U2-CLK-Pad13)
Routing:
- net /C10-28: track 110.8 -> 0.00 mm
- net /C7-38: track 84.7 -> 0.00 mm
- net /C7-36: track 80.4 -> 0.00 mm
- net +3V3: track 102.3 -> 22.0 mm
- net /ACCEL: track 79.9 -> 0.00 mm
- net /C10-11: track 75.1 -> 0.00 mm
- net /A_IN: track 74.7 -> 5.61 mm
- net /C10-34: track 127.0 -> 63.7 mm
- net /C7-28: track 68.3 -> 5.10 mm
- net unconnected-(J3-Pad66): track 0.00 -> 53.7 mm
- net /H_U: track 41.9 -> 0.00 mm
- net /SW3: track 31.3 -> 0.00 mm
- net Net-(SW2-B): track 19.6 -> 0.00 mm
- net /_LIN_S: track 18.2 -> 0.00 mm
- net Net-(JP1-A): track 9.19 -> 0.00 mm
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Other:
- board text removed: "0"
- board text removed: "Motor"
- board text removed: "|"

Commit message: 0417
Parts:
- removed S3, S4: TVGP01-G73BB, SamacSys_Parts:TVGP01G73BB
- added J4: RJ45_LED_Shielded, Connector_RJ:RJ45_Amphenol_RJHSE538X, F.Cu at (128.7, 68.4)
- added J6: JTAG, Connector_PinHeader_2.54mm:PinHeader_1x04_P2.54mm_Vertical, F.Cu at (148.1, 119.4)
- added R3: 5.1k, Resistor_SMD:R_0603_1608Metric_Pad0.98x0.95mm_HandSolder, F.Cu at (94.8, 88.9)
- added R4: 5.1k, Resistor_SMD:R_0603_1608Metric_Pad0.98x0.95mm_HandSolder, F.Cu at (94.8, 91.4)
- added R5: 5.1k, Resistor_SMD:R_0603_1608Metric_Pad0.98x0.95mm_HandSolder, F.Cu at (94.8, 93.9)
- added SW1: SW_SPDT, Connector_PinHeader_2.54mm:PinHeader_1x03_P2.54mm_Vertical, F.Cu at (77.8, 90.6)
- added SW2: SW_SPDT, Connector_PinHeader_2.54mm:PinHeader_1x03_P2.54mm_Vertical, F.Cu at (82.4, 90.6)
- added SW3: SW_SPDT, Connector_PinHeader_2.54mm:PinHeader_1x03_P2.54mm_Vertical, F.Cu at (87.1, 90.6)
- moved C1 30.0 mm to (156.6, 127.6)
- moved JP1 30.0 mm to (166.2, 128.1)
- moved R1 30.0 mm to (167.5, 130.6)
- moved R2 30.0 mm to (163.5, 131.2)
- moved U2 13.0 mm to (140.7, 125.3), turned to 0 degrees
- moved J2 6.20 mm to (159.0, 115.9)
- moved J1 2.47 mm to (171.0, 115.8)
Connections:
- J1 pad 24: /VCCIO0/1 -> VDD_3V3
- J1 pad 26: /VCCIO0/1 -> VDD_3V3
- J1 pad 29: /VCCIO6/7 -> VDD_3V3
- J1 pad 31: /VCCIO6/7 -> VDD_3V3
- J1 pad 34: /K7_IOT21A_40P -> /HIN_T
- J1 pad 38: /L7_IOT19A_40P -> /HIN_R
- J1 pad 42: /L10_IOT15A_40P -> /HIN_S
- J2 pad 2: /VCCIO2/3 -> VDD_3V3
- J2 pad 26: /J1_IOR33A_40P -> /H_U
- J2 pad 4: /VCCIO2/3 -> VDD_3V3
- J2 pad 46: /VDD_3V3 -> VDD_3V3
- J2 pad 48: /VDD_3V3 -> VDD_3V3
- J2 pad 50: /VDD_3V3 -> VDD_3V3
- J2 pad 6: /L2_IOR18A_40P -> /DIRECTION
- J3 pad 16: +3V3 -> VDD_3V3
- J3 pad 18: /5V -> /VDD_5V
- J3 pad 34: /_LIN_S -> /F5_IOT72A
- J3 pad 39: /C10-01 -> unconnected-(J3-Pad39)
- J3 pad 43: /D_IN -> unconnected-(J3-Pad43)
- J3 pad 56: /V -> unconnected-(J3-Pad56)
- J3 pad 62: /_LIN_T -> /G7_IOT68A
- J3 pad 63: /H_W -> /H1_IOB91A_40P
- J3 pad 64: /_LIN_R -> /H8_IOT66A
- J3 pad 66: unconnected-(J3-Pad66) -> /C10-28
- J3 pad 68: /C7-30 -> unconnected-(J3-Pad68)
- J3 pad 69: /H_V -> /G4_IOB89A_40P
- JP1 pad 2: +3V3 -> VDD_3V3
- PS1 pad 3: /5V -> /VDD_5V
- R1 pad 1: +3V3 -> VDD_3V3
- U2 pad 1: /C7-30 -> /C7-28
- U2 pad 10: /CS/SHDN -> /B2_IOB4A_40P
- U2 pad 11: /Din -> /C2_IOB4B_40P
- U2 pad 12: unconnected-(U2-Dout-Pad12) -> /F2_IOB26A_40P
- U2 pad 13: unconnected-(U2-CLK-Pad13) -> /F1_IOB26B_40P
- U2 pad 16: +3V3 -> VDD_3V3
- U2 pad 2: /C10-28 -> /C7-30
- U2 pad 3: /C10-34 -> /A_IN
- U2 pad 4: /C7-38 -> /C7-36
- U2 pad 5: /ACCEL -> /C7-38
- U2 pad 6: /C7-36 -> /ACCEL
- U2 pad 7: /A_IN -> /C10-28
- U2 pad 8: /C7-28 -> /C10-34
Routing:
- net /C10-34: track 63.7 -> 0.00 mm
- net unconnected-(J3-Pad66): track 53.7 -> 0.00 mm
- net /C10-28: track 0.00 -> 53.7 mm
- net /_LIN_T: track 23.5 -> 0.00 mm
- net /G7_IOT68A: track 0.00 -> 23.5 mm
- net /_LIN_R: track 22.7 -> 0.00 mm
- net /H8_IOT66A: track 0.00 -> 22.7 mm
- net VDD_3V3: track 0.00 -> 22.0 mm
- net +3V3: track 22.0 -> 0.00 mm
- net /VDD_5V: track 0.00 -> 18.3 mm
- net /5V: track 18.3 -> 0.00 mm
- net /A_IN: track 5.61 -> 0.00 mm
- net /C7-28: track 5.10 -> 0.00 mm
Other:
- board text added: "Tang Primer 25K - InverterKit2"
- board text removed: "I/O 1.8V"
- board text removed: "Tang Nano 9K - InverterKit2"

Commit message: 0418
Parts:
- added S1: TVGP01-G73BB, SamacSys_Parts:TVGP01G73BB, F.Cu at (175.1, 138.1)
- added S2: TVGP01-G73BB, SamacSys_Parts:TVGP01G73BB, F.Cu at (190.9, 138.2)
- J6: value JTAG -> Conn_01x04
- moved R4 80.2 mm to (167.5, 125.3), turned to 180 degrees
- moved SW3 70.1 mm to (132.8, 143.8)
- moved SW2 69.9 mm to (127.8, 143.8)
- moved SW1 69.5 mm to (122.6, 143.8)
- moved R3 66.8 mm to (153.7, 120.5), turned to 90 degrees
- moved R5 56.8 mm to (146.7, 117.1), turned to -90 degrees
- moved JP1 15.0 mm to (151.3, 126.1)
- moved R1 14.6 mm to (153.7, 126.1), turned to -90 degrees
- moved R2 9.94 mm to (153.7, 129.6), turned to -90 degrees
- moved J6 6.84 mm to (146.7, 112.7), turned to 90 degrees
- moved C1 5.69 mm to (151.3, 129.6), turned to -90 degrees
- moved J1 4.06 mm to (175.0, 116.2)
- moved J2 2.05 mm to (161.0, 116.2)
Connections:
- J1 pad 46: /K11_IOT11A -> /H_V
- J2 pad 26: /H_U -> /J1_IOR33A_40P
- J3 pad 17: /H_U -> /A11_IOL14A
- J3 pad 63: /H1_IOB91A_40P -> /E11_IOL3A
- J3 pad 69: /G4_IOB89A_40P -> /H_V
- U2 pad 7: /C10-28 -> /C10-34
- U2 pad 8: /C10-34 -> /C10-28
Routing:
- net /A11_IOL14A: track 0.00 -> 100.6 mm, vias 0 -> 1
- net VDD_3V3: track 22.0 -> 108.6 mm, vias 0 -> 1
- net /C10-34: track 0.00 -> 72.1 mm
- net /F5_IOT72A: track 0.00 -> 59.2 mm, vias 0 -> 1
- net /DIRECTION: track 0.00 -> 51.0 mm, vias 0 -> 1
- net GND: track 0.22 -> 27.0 mm, vias 4 -> 14
- net /B2_IOB4A_40P: track 0.00 -> 26.6 mm
- net /VDD_5V: track 18.3 -> 44.2 mm
- net /ACCEL: track 0.00 -> 25.8 mm
- net /C2_IOB4B_40P: track 0.00 -> 25.2 mm
- net /F2_IOB26A_40P: track 0.00 -> 23.9 mm
- net /L5_IOT63A: track 0.00 -> 22.7 mm, vias 0 -> 1
- net /F1_IOB26B_40P: track 0.00 -> 22.7 mm
- net /H_V: track 0.00 -> 22.3 mm, vias 0 -> 1
- net /H5_IOT61A: track 0.00 -> 21.8 mm, vias 0 -> 1
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Other:
- board size 81.5 x 99.9 mm -> 80.5 x 99.9 mm
- board text removed: "25"
- board text removed: "26"
- board text removed: "27"
- board text removed: "28"
- board text removed: "29"
- board text removed: "30"
- board text removed: "31/Dout"
- board text removed: "32/CLK"
- board text removed: "33"
- board text removed: "34"
- board text removed: "35"
- board text removed: "36"
- board text removed: "36/#LIN_T"
- board text removed: "37/#LIN_R"
- board text removed: "38/#LIN_S"
- board text removed: "39"
- board text removed: "40"
- board text removed: "41/H_V"
- board text removed: "42/H_W"
- board text removed: "48/CS SHDN"
- board text removed: "49/Din"
- board text removed: "51"
- board text removed: "53"
- board text removed: "54"
- board text removed: "55"
- board text removed: "56"
- board text removed: "57"
- board text removed: "63/H_U"
- board text removed: "68/D_IN"
- board text removed: "69/DIRECTION"
- board text removed: "70"
- board text removed: "71"
- board text removed: "72"
- board text removed: "73"
- board text removed: "74"
- board text removed: "75"
- board text removed: "76"
- board text removed: "77"
- board text removed: "80"
- board text removed: "81"
- board text removed: "82"
- board text removed: "83"
- board text removed: "84"
- board text removed: "85"
- board text removed: "86"
- board text removed: "[C-574SR-LF]"

Commit message: 0419
Parts:
- added U1: Pmod_CAN, Library:Pmod_CAN, F.Cu at (168.0, 66.1)
- moved R4 2.39 mm to (165.1, 125.2)
- moved SW2 2.22 mm to (128.3, 141.6)
- moved SW1 2.22 mm to (123.1, 141.6)
- moved SW3 2.22 mm to (133.3, 141.6)
Connections:
- SW1 pad 1: +3V3 -> VDD_3V3
- SW1 pad 2: unconnected-(SW1-B-Pad2) -> /L9_IOT31A_40P
- SW2 pad 1: +3V3 -> VDD_3V3
- SW2 pad 2: unconnected-(SW2-B-Pad2) -> /J8_IOT56A_40P
- SW3 pad 1: +3V3 -> VDD_3V3
- SW3 pad 2: /SW3 -> /F7_IOT58A_40P
Routing:
- net VDD_3V3: track 108.6 -> 204.3 mm
- net /L9_IOT31A_40P: track 0.00 -> 73.4 mm, vias 0 -> 1
- net /J8_IOT56A_40P: track 0.00 -> 66.1 mm, vias 0 -> 1
- net /F7_IOT58A_40P: track 0.00 -> 56.2 mm, vias 0 -> 1
- net /B11_IOL12A: track 0.00 -> 54.2 mm
- net /C11_IOL5A: track 0.00 -> 52.3 mm
- net /D11_IOL9A: track 0.00 -> 50.6 mm
- net /G11_IOT7A: track 0.00 -> 49.0 mm
- net Net-(U1-CAN_L): track 0.00 -> 12.0 mm
- net Net-(U1-CAN_H): track 0.00 -> 10.2 mm
- net /C10-28: track 65.9 -> 72.8 mm
- net /C10-34: track 72.1 -> 76.0 mm
- net GND: track 27.0 -> 28.7 mm, vias 14 -> 11
- net /E8_READY: track 9.36 -> 10.9 mm
- net /ACCEL: track 25.8 -> 25.0 mm

Commit message: 0421
Parts:
- added R6: 5.1k, Resistor_SMD:R_0603_1608Metric_Pad0.98x0.95mm_HandSolder, F.Cu at (137.7, 77.0)
- added R7: 5.1k, Resistor_SMD:R_0603_1608Metric_Pad0.98x0.95mm_HandSolder, F.Cu at (138.8, 57.1)
- added REF**: TestPoint_Pad_2.0x2.0mm, TestPoint:TestPoint_Pad_2.0x2.0mm, F.Cu at (123.1, 140.8)
- added REF**: TestPoint_Pad_2.0x2.0mm, TestPoint:TestPoint_Pad_2.0x2.0mm, F.Cu at (128.3, 140.8)
- added REF**: TestPoint_Pad_2.0x2.0mm, TestPoint:TestPoint_Pad_2.0x2.0mm, F.Cu at (133.3, 140.8)
- added REF**: TestPoint_Pad_2.0x2.0mm, TestPoint:TestPoint_Pad_2.0x2.0mm, F.Cu at (123.1, 151.4)
- added REF**: TestPoint_Pad_2.0x2.0mm, TestPoint:TestPoint_Pad_2.0x2.0mm, F.Cu at (128.3, 151.4)
- added REF**: TestPoint_Pad_2.0x2.0mm, TestPoint:TestPoint_Pad_2.0x2.0mm, F.Cu at (133.3, 151.4)
- moved SW1 1.92 mm to (123.1, 143.5)
- moved SW2 1.92 mm to (128.3, 143.5)
- moved SW3 1.92 mm to (133.3, 143.5)
- moved R3 1.28 mm to (152.8, 119.6), turned to 0 degrees
- moved R4 0.97 mm to (166.1, 125.3)
- moved JP1 0.23 mm to (151.3, 125.9)
Connections:
- J4 pad 10: unconnected-(J4-Pad10) -> Net-(J4-Pad10)
- J4 pad 11: unconnected-(J4-Pad11) -> /M0_D0_P
- J4 pad 12: unconnected-(J4-Pad12) -> Net-(J4-Pad12)
- J4 pad 9: unconnected-(J4-Pad9) -> /M0_D0_N
Routing:
- net VDD_3V3: track 204.3 -> 272.4 mm
- net /M0_D0_P: track 0.00 -> 66.5 mm, vias 0 -> 3
- net /M0_D0_N: track 0.00 -> 49.7 mm, vias 0 -> 2
- net Net-(J4-Pad10): track 0.00 -> 8.49 mm
- net /G11_IOT7A: track 49.0 -> 52.7 mm
- net /B11_IOL12A: track 54.2 -> 58.0 mm
- net /C11_IOL5A: track 52.3 -> 56.1 mm
- net /D11_IOL9A: track 50.6 -> 54.4 mm
- net Net-(J4-Pad12): track 0.00 -> 2.96 mm
- net /A11_IOL14A: track 100.6 -> 98.3 mm
- net /F7_IOT58A_40P: track 56.2 -> 55.4 mm
- net GND: vias 11 -> 33
Other:
- board text added: "CAN_H"
- board text added: "CAN_L"
- board text added: "VDD_5V"
- board text removed: "79"

Commit message: 0422
Parts:
- added J5: Conn_01x03, Connector_PinHeader_2.54mm:PinHeader_1x03_P2.54mm_Vertical, F.Cu at (160.9, 133.1)
- moved R4 6.54 mm to (161.8, 130.3), turned to 0 degrees
Connections:
- R4 pad 1: /E8_READY -> Net-(J5-Pin_1)
Routing:
- net /E8_READY: track 10.6 -> 24.2 mm
- net VDD_3V3: track 272.4 -> 277.6 mm
- net /F7_IOT58A_40P: track 55.4 -> 59.2 mm
- net /J8_IOT56A_40P: track 66.5 -> 70.1 mm
- net /L9_IOT31A_40P: track 73.4 -> 76.4 mm
- net Net-(J5-Pin_1): track 0.00 -> 2.80 mm
- net GND: vias 33 -> 34
Other:
- board text added: "Ready"
- board text added: "TCK"
- board text added: "TDI"
- board text added: "TDO"
- board text added: "TMS"
- board text added: "VDD_3V3"

Commit message: 0423
Parts:
- added G***: LOGO, footprints:kamo20, F.Cu at (162.2, 88.8)
Other:
- board size 80.5 x 99.9 mm -> 79.2 x 99.9 mm
