File: TangPrimer25K_brushless.kicad_pcb (KiCad board)
At the start: 2 copper layers, 79.2 x 99.9 mm, 30 parts, among them J1 DF40C-60DS-0.4V_51_, J2 DF40C-60DS-0.4V_51_, J3 Nucleo_F302R8, J4 RJ45_LED_Shielded, J5 Conn_01x03, J6 Conn_01x04, SW1 SW_SPDT, SW2 SW_SPDT, SW3 SW_SPDT, U1 Pmod_CAN, U2 MCP3008

Commit message: 0911
Parts:
- removed U1: Pmod_CAN, Library:Pmod_CAN
- added C2: 0.1u, Capacitor_SMD:C_0603_1608Metric_Pad1.08x0.95mm_HandSolder, F.Cu at (149.2, 63.4)
- added C3: 10u, Capacitor_SMD:C_0603_1608Metric_Pad1.08x0.95mm_HandSolder, F.Cu at (155.1, 67.2)
- added C4: 4.7n, Capacitor_SMD:C_0603_1608Metric_Pad1.08x0.95mm_HandSolder, F.Cu at (143.4, 74.0)
- added D4: SM24CANB-02HTG, samacsys:SM24CANB02HTG, F.Cu at (140.0, 60.7)
- added IC2: TJA1441AT, samacsys:SOIC127P600X175-8N, F.Cu at (149.2, 67.8)
- added L1: SDCW3216-2-222TF, samacsys:SDCW32162222TF, F.Cu at (140.4, 67.8)
- added R11: 4.7k, Resistor_SMD:R_0603_1608Metric_Pad0.98x0.95mm_HandSolder, F.Cu at (147.3, 71.6)
- added R13: 60.4, Resistor_SMD:R_0603_1608Metric_Pad0.98x0.95mm_HandSolder, F.Cu at (140.0, 71.2)
- added R14: 60.4, Resistor_SMD:R_0603_1608Metric_Pad0.98x0.95mm_HandSolder, F.Cu at (139.9, 64.4)
- added R8: 4.7k, Resistor_SMD:R_0603_1608Metric_Pad0.98x0.95mm_HandSolder, F.Cu at (152.9, 71.6)
- added R9: 4.7k, Resistor_SMD:R_0603_1608Metric_Pad0.98x0.95mm_HandSolder, F.Cu at (152.0, 63.4)
- added TP1: TestPoint, TestPoint:TestPoint_Pad_D1.5mm, F.Cu at (123.7, 126.0)
- moved R6 4.94 mm to (133.0, 78.5)
- moved R7 4.60 mm to (134.4, 58.4), turned to 0 degrees
- moved J4 3.00 mm to (128.7, 71.4)
Connections:
- J1 pad 43: /G10_IOT7B -> /DIRECTION
- J2 pad 6: /DIRECTION -> /L2_IOR18A_40P
- J4 pad 11: /M0_D0_P -> /H10_IOT3B_S2
- J4 pad 9: /M0_D0_N -> /J10_IOT1B_40P
Routing:
- net /M0_D0_P: track 66.5 -> 0.00 mm, vias 3 -> 0
- net /G11_IOT7A: track 52.7 -> 0.00 mm
- net /M0_D0_N: track 49.7 -> 0.00 mm, vias 2 -> 0
- net /B11_IOL12A: track 58.0 -> 31.3 mm
- net /C11_IOL5A: track 56.1 -> 33.3 mm
- net /D11_IOL9A: track 54.4 -> 35.3 mm
- net Net-(D4-Pad2): track 10.2 -> 29.1 mm, vias 0 -> 1
- net Net-(C4-Pad1): track 0.00 -> 13.8 mm, vias 0 -> 2
- net /DIRECTION: track 50.9 -> 37.9 mm
- net VDD_3V3: track 277.6 -> 285.7 mm, vias 1 -> 2
- net /VDD_5V: track 44.2 -> 52.1 mm
- net /A11_IOL14A: track 98.3 -> 105.3 mm
- net /ACCEL: track 25.0 -> 31.6 mm
- net Net-(IC2-CANH): track 0.00 -> 4.83 mm
- net Net-(IC2-CANL): track 0.00 -> 4.82 mm
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
Commit message: 0912
Parts:
- moved R7 1.52 mm to (134.4, 56.9)
- moved R6 1.25 mm to (133.0, 79.7)
Routing:
- net /H10_IOT3B_S2: track 0.00 -> 89.9 mm, vias 0 -> 1
- net /J10_IOT1B_40P: track 0.00 -> 62.6 mm
- net /VDD_5V: track 52.1 -> 101.7 mm, vias 0 -> 3
- net /B11_IOL12A: track 31.3 -> 64.7 mm
- net /D11_IOL9A: track 35.3 -> 66.2 mm
- net /C11_IOL5A: track 33.3 -> 60.3 mm
- net /A11_IOL14A: track 105.3 -> 102.0 mm
- net VDD_3V3: track 285.7 -> 284.1 mm
- net Net-(J4-Pad12): track 2.54 -> 4.07 mm
- net Net-(J4-Pad10): track 6.90 -> 8.14 mm
- net /DIRECTION: track 37.9 -> 38.5 mm
- net GND: vias 28 -> 38
Other:
- board text added: "Tang Primer 25K - InverterKit2 v0.2"
- board text removed: "Tang Primer 25K - InverterKit2"

Commit message: 1023
Parts:
- added J8: Conn_01x02, Connector_PinHeader_2.54mm:PinHeader_1x02_P2.54mm_Vertical, F.Cu at (123.1, 113.9)
- moved C4 1.24 mm to (142.5, 73.2), turned to 180 degrees
- moved R7 0.76 mm to (134.4, 57.7)
- moved C2 0.25 mm to (149.5, 63.4)
- moved R9 0.18 mm to (152.1, 63.4)
Connections:
- IC2 pad 5: +3V3 -> VDD_3V3
Routing:
- net VDD_3V3: track 284.1 -> 306.2 mm, vias 2 -> 1
- net Net-(J4-Pad12): track 4.07 -> 3.31 mm
- net /VDD_5V: track 101.7 -> 101.1 mm
- net Net-(D4-Pad2): track 29.1 -> 28.6 mm
- net GND: vias 38 -> 41
Other:
- board text added: "Tang Primer 25K - InverterKit2 v0.3"
- board text removed: "Tang Primer 25K - InverterKit2 v0.2"
