File: TangPrimer25K_brushless.kicad_sch (KiCad schematic)
At the start: 14 parts, among them J1 DF40C-60DS-0.4V_51_, J2 DF40C-60DS-0.4V_51_, J3 Nucleo_F302R8, SW1 SW_SPDT, SW2 SW_SPDT, SW3 SW_SPDT, U2 MCP3008

Commit message: 0416
Connections:
- net L6_IOT23A_USB_P: now reaches J1.30
- net K6_IOT23B_USB_N: now reaches J1.32
- net J11_IOT1A_40P: now reaches J1.33
- net K7_IOT21A_40P: now reaches J1.34
- net J10_IOT1B_40P: now reaches J1.35
- net J7_IOT21B_40P: now reaches J1.36
- net H11_IOT3A_S1: now reaches J1.37
- net L7_IOT19A_40P: now reaches J1.38
- net H10_IOT3B_S2: now reaches J1.39
- net L8_IOT19B_40P: now reaches J1.40
- net G11_IOT7A: now reaches J1.41
- net L10_IOT15A_40P: now reaches J1.42
- net G10_IOT7B: now reaches J1.43
- net K10_IOT15B_40P: now reaches J1.44
- net K11_IOT11A: now reaches J1.46
- net D11_IOL9A: now reaches J1.47
- net L11_IOT11B: now reaches J1.48
- net D10_IOL9B: now reaches J1.49
- net C11_IOL5A: now reaches J1.51
- net E11_IOL3A: now reaches J1.52
- net C10_IOL5B: now reaches J1.53
- net E10_IOL3B: now reaches J1.54
- net B11_IOL12A: now reaches J1.55
- net A11_IOL14A: now reaches J1.56
- net B10_IOL12B: now reaches J1.57
- net A10_IOL14B: now reaches J1.58

Commit message: 0416
Parts:
- added J4: RJ45_LED_Shielded, Connector_RJ:RJ45_Amphenol_RJHSE538X, symbol Connector:RJ45_LED_Shielded
- added J6: Conn_01x04, Connector_PinHeader_2.54mm:PinHeader_1x04_P2.54mm_Vertical, symbol Connector_Generic:Conn_01x04
- added R3, R4, R5: 5.1k, Resistor_THT:R_Axial_DIN0207_L6.3mm_D2.5mm_P7.62mm_Horizontal, symbol Device:R
- added U1: Pmod_CAN, symbol New_Library:Pmod_CAN
- J1, J2: footprint DF40C-60DS-0.4V(51) -> Library:DF40C-60DS-0.4V_51_
Connections:
- net CS/SHDN is gone; now on net B2_IOB4A_40P: U2.10 (~{CS}/SHDN)
- net Din is gone; now on net C2_IOB4B_40P: U2.11 (Din)
- net VCCIO0/1 is gone; now on net VDD_3V3: J1.24, J1.26
- net VCCIO2/3 is gone; now on net VDD_3V3: J2.2, J2.4
- net VCCIO6/7 is gone; now on net VDD_3V3: J1.29, J1.31
- net +3V3: no longer J3.16 (Pin_16), JP1.2 (B), R1.1, U2.16 (Vdd)
- net 5V: no longer PS1.3 (VOUT)
- net A2_JTAG_TDO: now also J6.3 (Pin_3)
- net A3_JTAG_TDI: now also J6.4 (Pin_4)
- net B1_JTAG_TMS: now also J6.2 (Pin_2)
- net C10-11: no longer U2.1 (CH0)
- net C10-28: no longer J3.66
- net C1_JTAG_TCK: now also J6.1 (Pin_1), R5.1
- net C7-30: now also J3.68, U2.1 (CH0)
- net D8_RECONFIG: now also R3.2
- net E8_READY: now also R4.1
- net GND: now also J1.1, J1.15, J1.2, J1.27, J1.28, J1.45, J1.50, J1.59, J1.60, J2.1, J2.19, J2.29, J2.35, J2.41, J2.47, J2.53, J2.59, R5.2, U1.11 (GND), U1.5 (GND)
- net VDD_3V3: now also J3.16 (Pin_16), JP1.2 (B), R1.1, U2.16 (Vdd), R3.1, R4.2, U1.12 (Vcc), U1.6 (Vcc)
- net VDD_5V: now also PS1.3 (VOUT)
- net F2_IOB26A_40P: now reaches U2.12 (Dout)
- net F2_IOB26A_40P: now also J2.7
- net F1_IOB26B_40P: now reaches U2.13 (CLK)
- net F1_IOB26B_40P: now also J2.9
- net F7_IOT58A_40P: now reaches J1.11
- net F6_IOT58B_40P: now reaches J1.13
- net L9_IOT31A_40P: now reaches J1.3
- net K9_IOT31B_40P: now reaches J1.5
- net J8_IOT56A_40P: now reaches J1.7
- net K8_IOT56B_40P: now reaches J1.9
- net K1_IOR20A_40P: now reaches J2.10
- net A1_IOB24A_40P: now reaches J2.11
- net K2_IOR20B_40P: now reaches J2.12
- net J4_IOR22A_40P: now reaches J2.14
- net E1_IOB12B_40P: now reaches J2.15
- net K4_IOR22B_40P: now reaches J2.16
- net D1_IOB14B_40P: now reaches J2.17
- net G2_IOR24A_40P: now reaches J2.18
- net G1_IOR24B_40P: now reaches J2.20
- net L4_IOR31A_40P: now reaches J2.22
- net L3_IOR31B_40P: now reaches J2.24
- net J1_IOR33A_40P: now reaches J2.26
- net J2_IOR33B_40P: now reaches J2.28
- net B2_IOB4A_40P: now reaches J2.3
- net G4_IOB89A_40P: now reaches J2.30
- net M0_D3_P: now reaches J2.31
- net H4_IOB89B_40P: now reaches J2.32
- net M0_D3_N: now reaches J2.33
- net H1_IOB91A_40P: now reaches J2.34
- net H2_IOB91B_40P: now reaches J2.36
- net M0_D2_P: now reaches J2.37
- net M0_D2_N: now reaches J2.39
- net M0_CK_P: now reaches J2.43
- net M0_CK_N: now reaches J2.45
- net M0_D1_P: now reaches J2.49
- net C2_IOB4B_40P: now reaches J2.5
- net M0_D1_N: now reaches J2.51
- net M0_D0_P: now reaches J2.55
- net M0_D0_N: now reaches J2.57
- net L2_IOR18A_40P: now reaches J2.6
- net L1_IOR18B_40P: now reaches J2.8
- net C10-01: no longer names the net of J3.39
- new net: J4.4, U1.13 (CAN_H)
- new net: J4.5, U1.14 (CAN_L)
- no-connect marks 47 -> 49
Other:
- moved on the sheet: C1, J1, J2, JP1, PS1, R1, R2, S3, S4, SW1, SW2, SW3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

Commit message: 0417
Parts:
- R3, R4, R5: footprint Resistor_THT:R_Axial_DIN0207_L6.3mm_D2.5mm_P7.62mm_Horizontal -> Resistor_SMD:R_0603_1608Metric_Pad0.98x0.95mm_HandSolder
- renumbered S4 to S1, S3 to S2
Connections:
- net 5V is gone; now on net VDD_5V: J3.18 (Pin_18)
- net H_V is gone; now on net G4_IOB89A_40P: J3.69
- net H_W is gone; now on net H1_IOB91A_40P: J3.63
- net J1_IOR33A_40P is gone; now on net H_U: J2.26
- net K7_IOT21A_40P is gone; now on net HIN_T: J1.34
- net L10_IOT15A_40P is gone; now on net HIN_S: J1.42
- net L2_IOR18A_40P is gone; now on net DIRECTION: J2.6
- net L7_IOT19A_40P is gone; now on net HIN_R: J1.38
- net _LIN_R is gone; now on net H8_IOT66A: J3.64
- net _LIN_S is gone; now on net F5_IOT72A: J3.34 (Pin_34)
- net _LIN_T is gone; now on net G7_IOT68A: J3.62
- net ACCEL: now also U2.6 (CH5); no longer U2.5 (CH4)
- net A_IN: now also U2.3 (CH2); no longer U2.7 (CH6)
- net C10-28: now also J3.66, U2.7 (CH6); no longer U2.2 (CH1)
- net C10-34: now also U2.8 (CH7); no longer U2.3 (CH2)
- net C7-28: now also U2.1 (CH0); no longer U2.8 (CH7)
- net C7-30: now also U2.2 (CH1); no longer J3.68, U2.1 (CH0)
- net C7-36: now also U2.4 (CH3); no longer U2.6 (CH5)
- net C7-38: now also U2.5 (CH4); no longer U2.4 (CH3)
- net D_IN: no longer names the net of J3.43
- net V: no longer names the net of J3.56
- no-connect marks 49 -> 50

Commit message: 0418
Connections:
- net A11_IOL14A: now also J3.17 (Pin_17)
- net B11_IOL12A: now also U1.10 (RxD)
- net C10-28: now also U2.8 (CH7); no longer U2.7 (CH6)
- net C10-34: now also U2.7 (CH6); no longer U2.8 (CH7)
- net C11_IOL5A: now also U1.9 (TxD)
- net D11_IOL9A: now also U1.8 (S)
- net E11_IOL3A: now also J3.63
- net G11_IOT7A: now also U1.7 (WS2812B)
- net G4_IOB89A_40P: no longer J3.69
- net H1_IOB91A_40P: no longer J3.63
- net H5_IOT61A: now also S1.3 (NO_1)
- net L5_IOT63A: now also S2.3 (NO_1)
- net H_U renamed J1_IOR33A_40P
- net J1_IOR33A_40P: no longer J3.17 (Pin_17)
- net K11_IOT11A renamed H_V
- net H_V: now also J3.69
Other:
- moved on the sheet: J3, J4, PS1, U1

Commit message: 0419
Parts:
- U1: footprint (none) -> Library:Pmod_CAN
Connections:
- net +3V3 is gone; now on net VDD_3V3: SW1.1 (A), SW2.1 (A), SW3.1 (A)
- net SW3 is gone; now on net F7_IOT58A_40P: SW3.2 (B)
- net J8_IOT56A_40P: now also SW2.2 (B)
- net L9_IOT31A_40P: now also SW1.2 (B)
Changed lines of the file:
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@@
 	(wire
 		(pts
+			(xy 99.695 64.77) (xy 124.46 64.77)
+		)
+		(stroke
+			(width 0)
+			(type default)
+		)
+	)
+	(wire
+		(pts
 			(xy 99.06 185.42) (xy 104.775 185.42)
 		)
@@
 	(wire
 		(pts
-			(xy 106.68 64.77) (xy 99.695 64.77)
-		)
-		(stroke
-			(width 0)
-			(type default)
-		)
-	)
-	(wire
-		(pts
 			(xy 219.075 116.205) (xy 212.09 116.205)
 		)
@@
 	(wire
 		(pts
-			(xy 29.845 97.155) (xy 36.195 97.155)
+			(xy 29.845 99.695) (xy 36.83 99.695)
 		)
 		(stroke
@@
 	(wire
 		(pts
-			(xy 29.845 97.155) (xy 29.845 99.695)
-		)
-		(stroke
-			(width 0)
-			(type default)
-		)
-	)
-	(wire
-		(pts
 			(xy 250.19 45.72) (xy 250.19 50.165)
 		)
@@
 	(wire
 		(pts
-			(xy 76.835 100.33) (xy 70.485 100.33)
+			(xy 99.695 59.69) (xy 124.46 59.69)
 		)
 		(stroke
@@
 	(wire
 		(pts
-			(xy 219.075 93.345) (xy 212.09 93.345)
+			(xy 76.835 100.33) (xy 70.485 100.33)
 		)
 		(stroke
@@
 	(wire
 		(pts
-			(xy 38.1 190.5) (xy 40.64 190.5)
+			(xy 219.075 93.345) (xy 212.09 93.345)
 		)
 		(stroke
@@
 	(wire
 		(pts
-			(xy 105.41 95.25) (xy 99.695 95.25)
+			(xy 38.1 190.5) (xy 40.64 190.5)
 		)
 		(stroke
@@
 	(wire
 		(pts
-			(xy 186.055 113.665) (xy 189.23 113.665)
+			(xy 105.41 95.25) (xy 99.695 95.25)
 		)
 		(stroke
@@
 	(wire
 		(pts
-			(xy 140.97 72.39) (xy 142.24 72.39)
+			(xy 186.055 113.665) (xy 189.23 113.665)
 		)
 		(stroke
@@
 	(wire
 		(pts
-			(xy 106.68 59.69) (xy 99.695 59.69)
+			(xy 140.97 72.39) (xy 142.24 72.39)
 		)
 		(stroke
@@
 	(wire
 		(pts
+			(xy 99.695 54.61) (xy 124.46 54.61)
+		)
+		(stroke
+			(width 0)
+			(type default)
+		)
+	)
+	(wire
+		(pts
 			(xy 17.78 102.235) (xy 19.685 102.235)
 		)
@@
 	(wire
 		(pts
-			(xy 106.68 54.61) (xy 99.695 54.61)
-		)
-		(stroke
-			(width 0)
-			(type default)
-		)
-	)
-	(wire
-		(pts
 			(xy 19.685 88.9) (xy 17.78 88.9)
 		)
@@
 	(wire
 		(pts
-			(xy 36.195 94.615) (xy 29.845 94.615)
+			(xy 29.845 86.36) (xy 41.91 86.36)
 		)
 		(stroke
@@
 	(wire
 		(pts
-			(xy 29.845 94.615) (xy 29.845 86.36)
-		)
-		(stroke
-			(width 0)
-			(type default)
-		)
-	)
-	(wire
-		(pts
 			(xy 240.03 33.655) (xy 235.585 33.655)
 		)
@@
 		)
 	)
+	(label "SW2"
+		(at 124.46 59.69 0)
+		(fields_autoplaced yes)
+		(effects
+			(font
+				(size 1.27 1.27)
+			)
+			(justify left bottom)
+		)
+	)
 	(label "H_U"
 		(at 52.705 120.65 180)
@@
 		)
 	)
+	(label "SW3"
+		(at 124.46 64.77 0)
+		(fields_autoplaced yes)
+		(effects
+			(font
+				(size 1.27 1.27)
+			)
+			(justify left bottom)
+		)
+	)
 	(label "H_U"
 		(at 17.78 165.1 0)
@@
 		)
 	)
+	(label "SW1"
+		(at 124.46 54.61 0)
+		(fields_autoplaced yes)
+		(effects
+			(font
+				(size 1.27 1.27)
+			)
+			(justify left bottom)
+		)
+	)
 	(label "B1_JTAG_TMS"
 		(at 219.075 80.645 0)
@@
 		)
 	)
+	(label "SW1"
+		(at 36.83 99.695 180)
+		(fields_autoplaced yes)
+		(effects
+			(font
+				(size 1.27 1.27)
+			)
+			(justify right bottom)
+		)
+	)
 	(label "VDD_3V3"
 		(at 184.785 50.8 180)
@@
 		)
 	)
+	(label "SW2"
+		(at 41.91 86.36 180)
+		(fields_autoplaced yes)
+		(effects
+			(font
+				(size 1.27 1.27)
+			)
+			(justify right bottom)
+		)
+	)
 	(label "VIN12"
 		(at 41.91 172.72 0)
@@
 			)
 		)
-		(property "Value" "+3V3"
+		(property "Value" "VDD_3V3"
 			(at 17.78 64.77 0)
 			(effects
@@
 			)
 		)
-		(property "Footprint" ""
+		(property "Footprint" "Library:Pmod_CAN"
 			(at 161.29 146.685 0)
 			(effects

Commit message: 0421
Parts:
- added R6, R7: 5.1k, Resistor_SMD:R_0603_1608Metric_Pad0.98x0.95mm_HandSolder, symbol Device:R
Connections:
- net M0_D0_N: now also J4.9
- net M0_D0_P: now also J4.11
- net VDD_3V3: now also R6.1, R7.1
- net at J4.10: now also R6.2
- net at J4.12: now also R7.2

Commit message: 0422
Parts:
- added J5: Conn_01x03, Connector_PinHeader_2.54mm:PinHeader_1x03_P2.54mm_Vertical, symbol Connector_Generic:Conn_01x03
Connections:
- net E8_READY: now also J5.2 (Pin_2); no longer R4.1
- net GND: now also J5.3 (Pin_3)
- new net: J5.1 (Pin_1), R4.1
Other:
- moved on the sheet: R4
Changed lines of the file:
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@@
 	(wire
 		(pts
+			(xy 136.525 59.69) (xy 136.525 60.96)
+		)
+		(stroke
+			(width 0)
+			(type default)
+		)
+	)
+	(wire
+		(pts
 			(xy 99.695 64.77) (xy 124.46 64.77)
 		)
@@
 	(wire
 		(pts
+			(xy 136.525 68.58) (xy 136.525 69.85)
+		)
+		(stroke
+			(width 0)
+			(type default)
+		)
+	)
+	(wire
+		(pts
 			(xy 76.835 90.17) (xy 70.485 90.17)
 		)
@@
 	(wire
 		(pts
+			(xy 136.525 74.93) (xy 136.525 76.2)
+		)
+		(stroke
+			(width 0)
+			(type default)
+		)
+	)
+	(wire
+		(pts
 			(xy 270.51 31.115) (xy 273.05 31.115)
 		)
@@
 	(wire
 		(pts
-			(xy 140.97 72.39) (xy 142.24 72.39)
-		)
-		(stroke
-			(width 0)
-			(type default)
-		)
-	)
-	(wire
-		(pts
 			(xy 189.23 73.025) (xy 187.325 73.025)
 		)
@@
 	(wire
 		(pts
+			(xy 99.695 72.39) (xy 136.525 72.39)
+		)
+		(stroke
+			(width 0)
+			(type default)
+		)
+	)
+	(wire
+		(pts
 			(xy 217.17 75.565) (xy 217.17 52.705)
 		)
@@
 	(wire
 		(pts
-			(xy 99.695 72.39) (xy 133.35 72.39)
-		)
-		(stroke
-			(width 0)
-			(type default)
-		)
-	)
-	(wire
-		(pts
 			(xy 99.06 177.8) (xy 101.6 177.8)
 		)
@@
 	)
 	(symbol
+		(lib_id "Connector_Generic:Conn_01x03")
+		(at 141.605 72.39 0)
+		(unit 1)
+		(exclude_from_sim no)
+		(in_bom yes)
+		(on_board yes)
+		(dnp no)
+		(fields_autoplaced yes)
+		(property "Reference" "J5"
+			(at 144.78 71.1199 0)
+			(effects
+				(font
+					(size 1.27 1.27)
+				)
+				(justify left)
+			)
+		)
+		(property "Value" "Conn_01x03"
+			(at 144.78 73.6599 0)
+			(effects
+				(font
+					(size 1.27 1.27)
+				)
+				(justify left)
+			)
+		)
+		(property "Footprint" "Connector_PinHeader_2.54mm:PinHeader_1x03_P2.54mm_Vertical"
+			(at 141.605 72.39 0)
+			(effects
+				(font
+					(size 1.27 1.27)
+				)
+				(hide yes)
+			)
+		)
+		(property "Datasheet" "~"
+			(at 141.605 72.39 0)
+			(effects
+				(font
+					(size 1.27 1.27)
+				)
+				(hide yes)
+			)
+		)
+		(property "Description" "Generic connector, single row, 01x03, script generated (kicad-library-utils/schlib/autogen/connector/)"
+			(at 141.605 72.39 0)
+			(effects
+				(font
+					(size 1.27 1.27)
+				)
+				(hide yes)
+			)
+		)
+		(pin "1"
+		)
+		(pin "2"
+		)
+		(pin "3"
+		)
+		(instances
+			(project "TangPrimer25K_brushless"
+				(path "/8aff725f-ee01-408d-a4eb-7fb705fecf00"
+					(reference "J5")
+					(unit 1)
+				)
+			)
+		)
+	)
+	(symbol
 		(lib_id "power:VCC")
 		(at 154.305 156.21 0)
@@
 	)
 	(symbol
+		(lib_name "GND_6")
+		(lib_id "power:GND")
+		(at 136.525 76.2 0)
+		(unit 1)
+		(exclude_from_sim no)
+		(in_bom yes)
+		(on_board yes)
+		(dnp no)
+		(fields_autoplaced yes)
+		(property "Reference" "#PWR023"
+			(at 136.525 82.55 0)
+			(effects
+				(font
+					(size 1.27 1.27)
+				)
+				(hide yes)
+			)
+		)
+		(property "Value" "GND"
+			(at 136.525 81.28 0)
+			(effects
+				(font
+					(size 1.27 1.27)
+				)
+			)
+		)
+		(property "Footprint" ""
+			(at 136.525 76.2 0)
+			(effects
+				(font
+					(size 1.27 1.27)
+				)
+				(hide yes)
+			)
+		)
+		(property "Datasheet" ""
+			(at 136.525 76.2 0)
+			(effects
+				(font
+					(size 1.27 1.27)
+				)
+				(hide yes)
+			)
+		)
+		(property "Description" "Power symbol creates a global label with name \"GND\" , ground"
+			(at 136.525 76.2 0)
+			(effects
+				(font
+					(size 1.27 1.27)
+				)
+				(hide yes)
+			)
+		)
+		(pin "1"
+		)
+		(instances
+			(project "TangPrimer25K_brushless"
+				(path "/8aff725f-ee01-408d-a4eb-7fb705fecf00"
+					(reference "#PWR023")
+					(unit 1)
+				)
+			)
+		)
+	)
+	(symbol
 		(lib_id "power:GND")
 		(at 112.395 182.88 0)
@@
 	(symbol
 		(lib_id "Device:R")
-		(at 137.16 72.39 90)
+		(at 136.525 64.77 180)
 		(unit 1)
 		(exclude_from_sim no)
@@
 		(dnp no)
 		(property "Reference" "R4"
-			(at 137.16 70.485 90)
+			(at 134.62 64.77 90)
 			(effects
 				(font
@@
 		)
 		(property "Value" "5.1k"
-			(at 137.16 72.39 90)
+			(at 136.525 64.77 90)
 			(effects
 				(font
@@
 		)
 		(property "Footprint" "Resistor_SMD:R_0603_1608Metric_Pad0.98x0.95mm_HandSolder"
-			(at 137.16 74.168 90)
+			(at 138.303 64.77 90)
 			(effects
 				(font
@@
 		)
 		(property "Datasheet" "~"
-			(at 137.16 72.39 0)
+			(at 136.525 64.77 0)
 			(effects
 				(font
@@
 		)
 		(property "Description" "Resistor"
-			(at 137.16 72.39 0)
+			(at 136.525 64.77 0)
 			(effects
 				(font
@@
 		(lib_name "+3V3_2")
 		(lib_id "power:+3V3")
-		(at 142.24 72.39 0)
+		(at 136.525 59.69 0)
 		(unit 1)
 		(exclude_from_sim no)
@@
 		(dnp no)
 		(property "Reference" "#PWR015"
-			(at 142.24 76.2 0)
+			(at 136.525 63.5 0)
 			(effects
 				(font
@@
 		)
 		(property "Value" "VDD_3V3"
-			(at 143.51 68.58 0)
+			(at 137.795 55.88 0)
 			(effects
 				(font
@@
 		)
 		(property "Footprint" ""
-			(at 142.24 72.39 0)
+			(at 136.525 59.69 0)
 			(effects
 				(font
@@
 		)
 		(property "Datasheet" ""
-			(at 142.24 72.39 0)
+			(at 136.525 59.69 0)
 			(effects
 				(font
@@
 		)
 		(property "Description" "Power symbol creates a global label with name \"+3V3\""
-			(at 142.24 72.39 0)
+			(at 136.525 59.69 0)
 			(effects
 				(font

Commit message: 0911
Parts:
- removed U1: Pmod_CAN, Library:Pmod_CAN, symbol New_Library:Pmod_CAN
- added C2: 0.1u, Capacitor_SMD:C_0603_1608Metric_Pad1.08x0.95mm_HandSolder, symbol Device:C
- added C3: 10u, Capacitor_SMD:C_0603_1608Metric_Pad1.08x0.95mm_HandSolder, symbol Device:C
- added C4: 4.7n, Capacitor_SMD:C_0603_1608Metric_Pad1.08x0.95mm_HandSolder, symbol Device:C
- added D4: SM24CANB-02HTG, samacsys:SM24CANB02HTG, symbol samacsys:SM24CANB-02HTG
- added IC2: TJA1441AT, samacsys:SOIC127P600X175-8N, symbol samacsys:TJA1441BT_0Z
- added L1: SDCW3216-2-222TF, samacsys:SDCW32162222TF, symbol samacsys:SDCW3216-2-222TF
- added R11, R8, R9: 4.7k, Resistor_SMD:R_0603_1608Metric_Pad0.98x0.95mm_HandSolder, symbol Device:R
- added R13, R14: 60.4, Resistor_SMD:R_0603_1608Metric_Pad0.98x0.95mm_HandSolder, symbol Device:R
- added TP1: TestPoint, TestPoint:TestPoint_Pad_D1.5mm, symbol Connector:TestPoint
Connections:
- net G10_IOT7B is gone; now on net DIRECTION: J1.43
- net ACCEL: now also TP1.1
- net B11_IOL12A: now also IC2.4 (RXD), R9.1
- net C11_IOL5A: now also IC2.1 (TXD), R8.1
- net D11_IOL9A: now also IC2.8 (S), R11.1
- net DIRECTION: no longer J2.6
- net GND: now also C2.1, C3.1, C4.2, D4.3, IC2.2 (GND), R11.2, R8.2, R9.2
- net H10_IOT3B_S2: now also J4.11
- net J10_IOT1B_40P: now also J4.9
- net M0_D0_N: no longer J4.9
- net M0_D0_P: no longer J4.11
- net VDD_5V: now also C2.2, C3.2, IC2.3 (VCC)
- net at J4.4: now also D4.2, L1.3, R13.1
- net at J4.5: now also D4.1, L1.2, R14.2
- new net: IC2.6 (CANL), L1.1
- new net: IC2.7 (CANH), L1.4
- new net: C4.1, R13.2, R14.1
- new net +3V3: IC2.5 (VIO)
- new net L2_IOR18A_40P: J2.6
Other:
- moved on the sheet: J3, J4, PS1, R3, R5, R6, R7
