File: TangPrimer25K_brushless.kicad_sch (KiCad schematic)
At the start: 34 parts, among them IC2 TJA1441AT, J1 DF40C-60DS-0.4V_51_, J2 DF40C-60DS-0.4V_51_, J3 Nucleo_F302R8, J4 RJ45_LED_Shielded, J5 Conn_01x03, J6 Conn_01x04, SW1 SW_SPDT, SW2 SW_SPDT, SW3 SW_SPDT, U2 MCP3008

Commit message: 1002
Connections:
- net +3V3 is gone; now on net VDD_3V3: IC2.5 (VIO)
Changed lines of the file:
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@@
 			)
 		)
-		(property "Value" "+3V3"
+		(property "Value" "VDD_3V3"
 			(at 166.37 168.91 0)
 			(effects

Commit message: 1023
Parts:
- added J8: Conn_01x02, Connector_PinHeader_2.54mm:PinHeader_1x02_P2.54mm_Vertical, symbol Connector_Generic:Conn_01x02
Connections:
- net VDD_3V3: now also J8.1 (Pin_1), J8.2 (Pin_2)
Changed lines of the file:
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@@
 	)
 	(junction
+		(at 136.525 60.325)
+		(diameter 0)
+		(color 0 0 0 0)
+	)
+	(junction
 		(at 257.81 45.72)
 		(diameter 0)
@@
 	)
 	(junction
+		(at 142.875 60.325)
+		(diameter 0)
+		(color 0 0 0 0)
+	)
+	(junction
 		(at 184.785 52.705)
 		(diameter 0)
@@
 	(wire
 		(pts
-			(xy 136.525 59.69) (xy 136.525 60.96)
+			(xy 136.525 59.69) (xy 136.525 60.325)
 		)
 		(stroke
@@
 	(wire
 		(pts
+			(xy 136.525 60.325) (xy 136.525 60.96)
+		)
+		(stroke
+			(width 0)
+			(type default)
+		)
+	)
+	(wire
+		(pts
 			(xy 189.23 111.125) (xy 186.055 111.125)
 		)
@@
 	(wire
 		(pts
+			(xy 136.525 60.325) (xy 142.875 60.325)
+		)
+		(stroke
+			(width 0)
+			(type default)
+		)
+	)
+	(wire
+		(pts
 			(xy 257.81 45.72) (xy 257.81 43.815)
 		)
@@
 	(wire
 		(pts
+			(xy 142.875 60.325) (xy 142.875 61.595)
+		)
+		(stroke
+			(width 0)
+			(type default)
+		)
+	)
+	(wire
+		(pts
 			(xy 107.315 87.63) (xy 107.315 89.535)
 		)
@@
 	(wire
 		(pts
+			(xy 142.875 59.055) (xy 142.875 60.325)
+		)
+		(stroke
+			(width 0)
+			(type default)
+		)
+	)
+	(wire
+		(pts
 			(xy 189.23 75.565) (xy 187.325 75.565)
 		)
@@
 					(unit 1)
 				)
+			)
+		)
+	)
+	(symbol
+		(lib_id "Connector_Generic:Conn_01x02")
+		(at 147.955 59.055 0)
+		(unit 1)
+		(exclude_from_sim no)
+		(in_bom yes)
+		(on_board yes)
+		(dnp no)
+		(fields_autoplaced yes)
+		(property "Reference" "J8"
+			(at 151.13 59.0549 0)
+			(effects
+				(font
+					(size 1.27 1.27)
+				)
+				(justify left)
+			)
+		)
+		(property "Value" "Conn_01x02"
+			(at 151.13 61.5949 0)
+			(effects
+				(font
+					(size 1.27 1.27)
+				)
+				(justify left)
+			)
+		)
+		(property "Footprint" "Connector_PinHeader_2.54mm:PinHeader_1x02_P2.54mm_Vertical"
+			(at 147.955 59.055 0)
+			(effects
+				(font
+					(size 1.27 1.27)
+				)
+				(hide yes)
+			)
+		)
+		(property "Datasheet" "~"
+			(at 147.955 59.055 0)
+			(effects
+				(font
+					(size 1.27 1.27)
+				)
+				(hide yes)
+			)
+		)
+		(property "Description" "Generic connector, single row, 01x02, script generated (kicad-library-utils/schlib/autogen/connector/)"
+			(at 147.955 59.055 0)
+			(effects
+				(font
+					(size 1.27 1.27)
+				)
+				(hide yes)
+			)
+		)
+		(pin "1"
+		)
+		(pin "2"
+		)
+		(instances
+			(project "TangPrimer25K_brushless"
+				(path "/8aff725f-ee01-408d-a4eb-7fb705fecf00"
+					(reference "J8")
+					(unit 1)
+				)
